Commit message: Fix bbot_description

File: bbot_description/urdf/bbot_base/bbot_base.urdf.xacro (robot description, xacro)
@@ -152,9 +152,9 @@
       </collision>
       <inertial>
-        <origin rpy="${radians(90)} 0 0" />
+        <origin rpy="0 0 0" />
         <mass value="${wheel_mass}" />
-        <inertia ixx="${(3 * wheel_radius * wheel_radius + wheel_width * wheel_width) * wheel_mass / 2}" ixy="0.0" ixz="0.0"
+        <inertia ixx="${(3 * wheel_radius * wheel_radius + wheel_width * wheel_width) * wheel_mass / 12}" ixy="0.0" ixz="0.0"
                  iyy="${wheel_radius * wheel_radius * wheel_mass / 2}" iyz="0.0"
-                 izz="${(3 * wheel_radius * wheel_radius + wheel_width * wheel_width) * wheel_mass / 2}" />
+                 izz="${(3 * wheel_radius * wheel_radius + wheel_width * wheel_width) * wheel_mass / 12}" />
       </inertial>
     </link>

File: bbot_description/urdf/bbot_base/bbot_base_gazebo.urdf.xacro (robot description, xacro)
@@ -3,7 +3,5 @@
   <xacro:macro name="bbot_base_wheel_gazebo" params="prefix">
     <gazebo reference="base_${prefix}_wheel">
-      <mu1>1</mu1>
-      <mu2>0.7</mu2>
-      <fdir1>1 0 0</fdir1>
+      <minDepth>0.001</minDepth>
       <material>Gazebo/Black</material>
     </gazebo>
@@ -20,5 +18,5 @@
         <rightFrontJoint>base_fr_wheel_joint</rightFrontJoint>
         <leftRearJoint>base_rl_wheel_joint</leftRearJoint>
-        <rightRearJoint>base_fr_wheel_joint</rightRearJoint>
+        <rightRearJoint>base_rr_wheel_joint</rightRearJoint>
         <wheelSeparation>${2 * wheel_y}</wheelSeparation>
         <wheelDiameter>${2 * wheel_radius}</wheelDiameter>
@@ -35,5 +33,5 @@
     </gazebo>
     <gazebo reference="laser">
-      <sensor type="ray" name="laser">
+      <sensor type="gpu_ray" name="laser">
         <visualize>true</visualize>
         <update_rate>10</update_rate>
@@ -56,5 +54,5 @@
           </noise>
         </ray>
-        <plugin name="laser" filename="libgazebo_ros_laser.so">
+        <plugin name="laser" filename="libgazebo_ros_gpu_laser.so">
           <topicName>/scan_raw</topicName>
           <frameName>laser</frameName>
